File: hardware/ELV1/ELV1.kicad_pcb (KiCad board)
At the start: 2 copper layers, 97.3 x 75 mm, 141 parts, among them J1 15VAC Transformer out, J2 Top Panel, J3 FAN OUT, J4 Front Panel, J5 power in (inside), J6 Program Pins, J7 power in (outside), J8 power in (outside) for batter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, Q1 IRLML6344TRPBF, Q2 IRF4905, Q3 IRLML6344TRPBF, U1 TL431DBV, U10 TPS54302, U11 AP2112K-3.3, U2 LM358, U3 LM358, U4 LTV-817S, U5 LM2596S-12, U7 ADS1115IDGS, U8 STM32G030F6Px, U9 LM7815_TO220, Y1 8mHz

Commit message: Reorganize hardware: rename Electronic Load to ELV1, add ELV1-revision and KiCad libraries
- Move the KiCad project into hardware/ELV1/ and rename its files from 'Electronic Load' to 'ELV1'
- Add the ELV1 revision board as hardware/ELV1-revision/
- Add custom symbol and footprint libraries under hardware/libraries/
- Update library references to the renamed libraries (my-NMOS -> myNMOS, myNTC:Untitled -> myNTC:NTC)
- Ignore KiCad backup and local state files

Co-Authored-By: Claude Opus 5.5 <noreply@anthropic.com>
Parts:
- TH1: footprint myNTC:Untitled -> myNTC:NTC
