File: hardware/ELV1/ELV1.kicad_sch (KiCad schematic)
At the start: 152 parts, among them J1 15VAC Transformer out, J2 Top Panel, J3 FAN OUT, J4 Front Panel, J5 power in (inside), J6 Program Pins, J7 power in (outside), J8 power in (outside for batteri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, Q1 IRLML6344TRPBF, Q2 IRF4905, Q3 IRLML6344TRPBF, Q4 IRF4905, Q5 BC337, U1 IRFP260NPBF, U10 TPS54302, U11 AP2112K-3.3, U12 IRFP260NPBF, U13 IRFP260NPBF, U2 LM358, U3 LM358, U4 LTV-817S, U5 LM2596S-12, U6 IRFP260NPBF, U7 ADS1115IDGS, U8 STM32G030F6Px, U9 LM7815_TO220, Y1 8mHz

Commit message: Reorganize hardware: rename Electronic Load to ELV1, add ELV1-revision and KiCad libraries
- Move the KiCad project into hardware/ELV1/ and rename its files from 'Electronic Load' to 'ELV1'
- Add the ELV1 revision board as hardware/ELV1-revision/
- Add custom symbol and footprint libraries under hardware/libraries/
- Update library references to the renamed libraries (my-NMOS -> myNMOS, myNTC:Untitled -> myNTC:NTC)
- Ignore KiCad backup and local state files

Co-Authored-By: Claude Opus 5.5 <noreply@anthropic.com>
Parts:
- TH1: footprint myNTC:Untitled -> myNTC:NTC
- U1, U12, U13, U6: symbol my-NMOS:IRFP260NPBF -> myNMOS:IRFP260NPBF
