File: hardware/ELV1-revision/ELV1 revision.kicad_sch (KiCad schematic)
At the start: 228 parts, among them J1 15VAC 30VA Transformer out, J10 PROGRAM PINS, J2 FAN1, J3 FAN2, J4 Conn_02x10_Odd_Even, J5 DS18B20, J6 power in (outside), J7 power in (outside), Q1 IRLML6344TRPBF, Q2 IRLML6344TRPBF, Q3 IRLML6344TRPBF, Q4 IRLML6344TRPBF, Q5 IRLML6344TRPBF, Q6 IRLML6344TRPBF, SW3 SW_Push, U10 IRFB4110PBF, U12 SRV05-4, U13 LTV-817S, U15 CH340G, U16 SY6280AAC, U17 TPS54302, U2 MCP4725xxx-xCH, U20 STM32G071CBT6, U21 ADS1115IDGS, U3 AP2112K-3.3, U4 OPA2197xD, U6 TPS54302, U7 IRFP260NPBF, U8 IRFP260NPBF, U9 ADS1115IDGS, Y1 12MHZ CRYSTAL, Y2 ABM7-8.000MHZ-D2Y-T

Commit message: ELV1 revision: J4 footprint JST PUD -> JST PHD (B20B-PHDSS), same pad grid
Co-Authored-By: Claude Opus 5.5 <noreply@anthropic.com>
Parts:
- J4: footprint Connector_JST:JST_PUD_B20B-PUDSS_2x10_P2.00mm_Vertical -> Connector_JST:JST_PHD_B20B-PHDSS_2x10_P2.00mm_Vertical
Changed lines of the file:
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@@
 			)
 		)
-		(property "Footprint" "Connector_JST:JST_PUD_B20B-PUDSS_2x10_P2.00mm_Vertical"
+		(property "Footprint" "Connector_JST:JST_PHD_B20B-PHDSS_2x10_P2.00mm_Vertical"
 			(at 295.91 185.42 0)
 			(hide yes)

Commit message: Revert J4 footprint change (connector stays KLS PHB 2.0); note ELV1 temporary X-cap bleeder
This reverts commit 97f4282.

Co-Authored-By: Claude Opus 5.5 <noreply@anthropic.com>
Parts:
- J4: footprint Connector_JST:JST_PHD_B20B-PHDSS_2x10_P2.00mm_Vertical -> Connector_JST:JST_PUD_B20B-PUDSS_2x10_P2.00mm_Vertical
Changed lines of the file:
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@@
 			)
 		)
-		(property "Footprint" "Connector_JST:JST_PHD_B20B-PHDSS_2x10_P2.00mm_Vertical"
+		(property "Footprint" "Connector_JST:JST_PUD_B20B-PUDSS_2x10_P2.00mm_Vertical"
 			(at 295.91 185.42 0)
 			(hide yes)
