File: hardware/ELV1-revision/ELV1 revision.kicad_sch (KiCad schematic)
At the start: 228 parts, among them J1 15VAC 30VA Transformer out, J10 PROGRAM PINS, J2 FAN1, J3 FAN2, J4 Conn_02x10_Odd_Even, J5 DS18B20, J6 power in (outside), J7 power in (outside), Q1 IRLML6344TRPBF, Q2 IRLML6344TRPBF, Q3 IRLML6344TRPBF, Q4 IRLML6344TRPBF, Q5 IRLML6344TRPBF, Q6 IRLML6344TRPBF, SW3 SW_Push, U10 IRFB4110PBF, U12 SRV05-4, U13 LTV-817S, U15 CH340G, U16 SY6280AAC, U17 TPS54302, U2 MCP4725xxx-xCH, U20 STM32G071CBT6, U21 ADS1115IDGS, U3 AP2112K-3.3, U4 OPA2197xD, U6 TPS54302, U7 IRFP260NPBF, U8 IRFP260NPBF, U9 ADS1115IDGS, Y1 12MHZ CRYSTAL, Y2 ABM7-8.000MHZ-D2Y-T

Commit message: ELV1 revision: H18 - R116/R117 VMS-R100 parallel to R18/R19 (0.05R per channel), R2 22k
Setpoint full scale stays ~12 A total; ADS #1 PGA moves to +/-0.512 V.
Firmware guide and pin plan updated.

Co-Authored-By: Claude Opus 5.5 <noreply@anthropic.com>
Parts:
- added R116, R117: 0.1R VMS-R100, Resistor_SMD:R_2512_6332Metric_Pad1.40x3.35mm_HandSolder, symbol Device:R_Small
- R18, R19: value 0.1R SHUNT RESISTOR -> 0.1R VMS-R100
- R2: value 10K -> 22K
Connections:
- net GND: now also R116.2, R117.2
- net at NT3.2, R19.1, U8.3 (S): now also R117.1
- net at NT1.2, R18.1, U7.3 (S): now also R116.1
